File: 18650-14s-12p.kicad_pcb (KiCad board)
At the start: 2 copper layers, 250 x 251 mm, 87 parts, among them J1 Conn_01x14, J2 Conn_01x07

Commit message: Updated to 13s-12p
Parts:
- removed F10, F11, F12, F13, F14, F15, F16, F17, F18, F19, F20, F21, F22, F23, F24, F25, F26, F27, F28, F29, F30, F31, F32, F33, F34, F35, F36, F37, F38, F39, F40, F41, F42, F43, F44, F45, F46, F8, F9: Fuse, Fuse:pcbfuse_4a
- added B100: BatterySpring, Battery:batteryspring, F.Cu at (183.0, 163.0)
- added B101: BatterySpring, Battery:batteryspring, F.Cu at (203.0, 163.0)
- added B102: BatterySpring, Battery:batteryspring, F.Cu at (223.0, 163.0)
- added B103: BatterySpring, Battery:batteryspring, F.Cu at (243.0, 164.5)
- added B104: BatterySpring, Battery:batteryspring, F.Cu at (263.0, 163.0)
- added B105: BatterySpring, Battery:batteryspring, F.Cu at (23.0, 183.5)
- added B106: BatterySpring, Battery:batteryspring, F.Cu at (43.0, 183.0)
- added B107: BatterySpring, Battery:batteryspring, F.Cu at (63.0, 183.0)
- added B108: BatterySpring, Battery:batteryspring, F.Cu at (83.0, 183.0)
- added B109: BatterySpring, Battery:batteryspring, F.Cu at (103.0, 183.0)
- added B110: BatterySpring, Battery:batteryspring, F.Cu at (123.0, 183.0)
- added B111: BatterySpring, Battery:batteryspring, F.Cu at (143.0, 183.0)
- added B112: BatterySpring, Battery:batteryspring, F.Cu at (163.0, 183.0)
- added B113: BatterySpring, Battery:batteryspring, F.Cu at (183.0, 183.0)
- added B114: BatterySpring, Battery:batteryspring, F.Cu at (202.7, 183.1)
- added B115: BatterySpring, Battery:batteryspring, F.Cu at (223.0, 183.0)
- added B116: BatterySpring, Battery:batteryspring, F.Cu at (242.8, 183.1)
- added B117: BatterySpring, Battery:batteryspring, F.Cu at (263.0, 183.0)
- added B118: BatterySpring, Battery:batteryspring, F.Cu at (23.0, 203.0)
- added B119: BatterySpring, Battery:batteryspring, F.Cu at (42.7, 203.5)
- added B120: BatterySpring, Battery:batteryspring, F.Cu at (63.0, 203.0)
- added B121: BatterySpring, Battery:batteryspring, F.Cu at (83.0, 203.0)
- added B122: BatterySpring, Battery:batteryspring, F.Cu at (103.0, 203.0)
- added B123: BatterySpring, Battery:batteryspring, F.Cu at (123.2, 203.2)
- added B124: BatterySpring, Battery:batteryspring, F.Cu at (142.7, 202.7)
- added B125: BatterySpring, Battery:batteryspring, F.Cu at (162.8, 202.9)
- added B126: BatterySpring, Battery:batteryspring, F.Cu at (183.0, 203.0)
- added B127: BatterySpring, Battery:batteryspring, F.Cu at (203.0, 203.0)
- added B128: BatterySpring, Battery:batteryspring, F.Cu at (223.0, 203.0)
- added B129: BatterySpring, Battery:batteryspring, F.Cu at (243.0, 203.0)
- added B130: BatterySpring, Battery:batteryspring, F.Cu at (263.0, 203.0)
- added B131: BatterySpring, Battery:batteryspring, F.Cu at (23.0, 223.0)
- added B132: BatterySpring, Battery:batteryspring, F.Cu at (43.0, 223.0)
- added B133: BatterySpring, Battery:batteryspring, F.Cu at (63.0, 223.0)
- added B134: BatterySpring, Battery:batteryspring, F.Cu at (83.0, 223.0)
- added B135: BatterySpring, Battery:batteryspring, F.Cu at (103.0, 223.0)
- added B136: BatterySpring, Battery:batteryspring, F.Cu at (123.0, 223.0)
- added B137: BatterySpring, Battery:batteryspring, F.Cu at (143.0, 223.0)
- added B138: BatterySpring, Battery:batteryspring, F.Cu at (163.0, 223.0)
- added B139: BatterySpring, Battery:batteryspring, F.Cu at (183.0, 223.0)
- added B140: BatterySpring, Battery:batteryspring, F.Cu at (203.0, 223.0)
- added B141: BatterySpring, Battery:batteryspring, F.Cu at (223.0, 223.0)
- added B142: BatterySpring, Battery:batteryspring, F.Cu at (243.0, 223.0)
- added B143: BatterySpring, Battery:batteryspring, F.Cu at (263.0, 223.0)
- added B144: BatterySpring, Battery:batteryspring, F.Cu at (23.0, 243.0)
- added B145: BatterySpring, Battery:batteryspring, F.Cu at (43.0, 243.0)
- added B146: BatterySpring, Battery:batteryspring, F.Cu at (63.0, 243.0)
- added B147: BatterySpring, Battery:batteryspring, F.Cu at (83.0, 243.0)
- added B148: BatterySpring, Battery:batteryspring, F.Cu at (103.0, 243.0)
- added B149: BatterySpring, Battery:batteryspring, F.Cu at (123.0, 243.0)
- added B150: BatterySpring, Battery:batteryspring, F.Cu at (143.0, 243.0)
- added B151: BatterySpring, Battery:batteryspring, F.Cu at (163.0, 243.0)
- added B152: BatterySpring, Battery:batteryspring, F.Cu at (183.0, 243.0)
- added B153: BatterySpring, Battery:batteryspring, F.Cu at (203.0, 243.0)
- added B154: BatterySpring, Battery:batteryspring, F.Cu at (223.0, 243.0)
- added B155: BatterySpring, Battery:batteryspring, F.Cu at (243.0, 243.0)
- added B156: BatterySpring, Battery:batteryspring, F.Cu at (263.0, 243.0)
- added B40: BatterySpring, Battery:batteryspring, F.Cu at (23.1, 83.1)
- added B41: BatterySpring, Battery:batteryspring, F.Cu at (43.0, 83.0)
- added B42: BatterySpring, Battery:batteryspring, F.Cu at (63.0, 83.0)
- added B43: BatterySpring, Battery:batteryspring, F.Cu at (83.0, 83.0)
- added B44: BatterySpring, Battery:batteryspring, F.Cu at (103.0, 83.0)
- added B45: BatterySpring, Battery:batteryspring, F.Cu at (123.0, 83.0)
- added B46: BatterySpring, Battery:batteryspring, F.Cu at (143.0, 83.0)
- added B47: BatterySpring, Battery:batteryspring, F.Cu at (163.0, 83.0)
- added B48: BatterySpring, Battery:batteryspring, F.Cu at (183.0, 83.0)
- added B49: BatterySpring, Battery:batteryspring, F.Cu at (203.0, 83.0)
- added B50: BatterySpring, Battery:batteryspring, F.Cu at (223.0, 83.0)
- added B51: BatterySpring, Battery:batteryspring, F.Cu at (243.0, 83.0)
- added B52: BatterySpring, Battery:batteryspring, F.Cu at (263.0, 83.0)
- added B53: BatterySpring, Battery:batteryspring, F.Cu at (23.0, 103.0)
- added B54: BatterySpring, Battery:batteryspring, F.Cu at (43.0, 103.0)
- added B55: BatterySpring, Battery:batteryspring, F.Cu at (63.0, 103.0)
- added B56: BatterySpring, Battery:batteryspring, F.Cu at (83.0, 103.0)
- added B57: BatterySpring, Battery:batteryspring, F.Cu at (103.0, 103.0)
- added B58: BatterySpring, Battery:batteryspring, F.Cu at (122.5, 103.0)
- added B59: BatterySpring, Battery:batteryspring, F.Cu at (143.0, 103.0)
- added B60: BatterySpring, Battery:batteryspring, F.Cu at (163.0, 103.0)
- added B61: BatterySpring, Battery:batteryspring, F.Cu at (183.0, 103.0)
- added B62: BatterySpring, Battery:batteryspring, F.Cu at (203.0, 103.0)
- added B63: BatterySpring, Battery:batteryspring, F.Cu at (223.0, 103.0)
- added B64: BatterySpring, Battery:batteryspring, F.Cu at (243.0, 103.0)
- added B65: BatterySpring, Battery:batteryspring, F.Cu at (263.0, 103.0)
- added B66: BatterySpring, Battery:batteryspring, F.Cu at (23.0, 123.0)
- added B67: BatterySpring, Battery:batteryspring, F.Cu at (43.0, 123.0)
- added B68: BatterySpring, Battery:batteryspring, F.Cu at (63.0, 123.0)
- added B69: BatterySpring, Battery:batteryspring, F.Cu at (83.0, 123.0)
- added B70: BatterySpring, Battery:batteryspring, F.Cu at (103.0, 123.0)
- added B71: BatterySpring, Battery:batteryspring, F.Cu at (123.0, 123.0)
- added B72: BatterySpring, Battery:batteryspring, F.Cu at (143.0, 123.0)
- added B73: BatterySpring, Battery:batteryspring, F.Cu at (163.0, 123.0)
- added B74: BatterySpring, Battery:batteryspring, F.Cu at (183.0, 123.0)
- added B75: BatterySpring, Battery:batteryspring, F.Cu at (203.0, 123.0)
- added B76: BatterySpring, Battery:batteryspring, F.Cu at (223.0, 123.0)
- added B77: BatterySpring, Battery:batteryspring, F.Cu at (243.0, 123.0)
- added B78: BatterySpring, Battery:batteryspring, F.Cu at (263.0, 123.0)
- added B79: BatterySpring, Battery:batteryspring, F.Cu at (23.0, 143.0)
- added B80: BatterySpring, Battery:batteryspring, F.Cu at (43.0, 143.0)
- added B81: BatterySpring, Battery:batteryspring, F.Cu at (63.0, 143.0)
- added B82: BatterySpring, Battery:batteryspring, F.Cu at (83.0, 143.0)
- added B83: BatterySpring, Battery:batteryspring, F.Cu at (103.0, 143.0)
- added B84: BatterySpring, Battery:batteryspring, F.Cu at (123.0, 143.0)
- added B85: BatterySpring, Battery:batteryspring, F.Cu at (143.0, 143.0)
- added B86: BatterySpring, Battery:batteryspring, F.Cu at (163.0, 143.0)
- added B87: BatterySpring, Battery:batteryspring, F.Cu at (183.0, 143.0)
- added B88: BatterySpring, Battery:batteryspring, F.Cu at (203.0, 143.0)
- added B89: BatterySpring, Battery:batteryspring, F.Cu at (223.0, 143.0)
- added B90: BatterySpring, Battery:batteryspring, F.Cu at (243.0, 143.0)
- added B91: BatterySpring, Battery:batteryspring, F.Cu at (263.0, 143.0)
- added B92: BatterySpring, Battery:batteryspring, F.Cu at (23.0, 163.0)
- added B93: BatterySpring, Battery:batteryspring, F.Cu at (43.0, 163.0)
- added B94: BatterySpring, Battery:batteryspring, F.Cu at (63.0, 163.0)
- added B95: BatterySpring, Battery:batteryspring, F.Cu at (83.0, 163.0)
- added B96: BatterySpring, Battery:batteryspring, F.Cu at (103.0, 163.0)
- added B97: BatterySpring, Battery:batteryspring, F.Cu at (123.0, 163.0)
- added B98: BatterySpring, Battery:batteryspring, F.Cu at (143.0, 163.0)
- added B99: BatterySpring, Battery:batteryspring, F.Cu at (163.0, 163.0)
- added REF**: MountingHole_3.5mm, MountingHole:MountingHole_3.5mm, F.Cu at (213.0, 73.0)
- added REF**: MountingHole_3.5mm, MountingHole:MountingHole_3.5mm, F.Cu at (213.0, 193.0)
- added REF**: MountingHole_3.5mm, MountingHole:MountingHole_3.5mm, F.Cu at (73.0, 193.0)
- added REF**: MountingHole_3.5mm, MountingHole:MountingHole_3.5mm, F.Cu at (73.0, 73.0)
- moved J2 186.2 mm to (189.5, 271.0), turned to 270 degrees
- moved J1 161.3 mm to (113.0, 271.1), turned to 90 degrees
- moved F1 145.1 mm to (113.0, 259.5), turned to 90 degrees
- moved F2 144.2 mm to (118.0, 259.5), turned to 90 degrees
- moved F7 143.9 mm to (144.0, 259.0), turned to 90 degrees
- moved F3 143.5 mm to (123.0, 259.5), turned to 90 degrees
- moved F4 143.2 mm to (128.5, 259.5), turned to 90 degrees
- moved F6 143.1 mm to (138.5, 259.0), turned to 90 degrees
- moved F5 142.6 mm to (133.5, 259.0), turned to 90 degrees
- moved B5 0.44 mm to (103.0, 23.0), turned to 180 degrees
- turned B11 to 180 degrees
- turned B13 to 180 degrees
- turned B16 to 180 degrees
- turned B18 to 180 degrees
- turned B20 to 180 degrees
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Connections:
- B11 pad 1: Net-(B11-Pad1) -> Net-(B10-Pad1)
- B12 pad 1: Net-(B12-Pad1) -> Net-(B103-Pad1)
- B13 pad 1: Net-(B13-Pad1) -> Net-(B103-Pad1)
- B14 pad 1: Net-(B14-Pad1) -> Net-(B1-Pad1)
- B15 pad 1: Net-(B15-Pad1) -> Net-(B106-Pad1)
- B16 pad 1: Net-(B16-Pad1) -> Net-(B106-Pad1)
- B17 pad 1: Net-(B17-Pad1) -> Net-(B108-Pad1)
- B18 pad 1: Net-(B18-Pad1) -> Net-(B108-Pad1)
- B19 pad 1: Net-(B19-Pad1) -> Net-(B110-Pad1)
- B2 pad 1: Net-(B2-Pad1) -> Net-(B106-Pad1)
- B20 pad 1: Net-(B20-Pad1) -> Net-(B110-Pad1)
- B21 pad 1: Net-(B21-Pad1) -> Net-(B100-Pad1)
- B22 pad 1: Net-(B22-Pad1) -> Net-(B100-Pad1)
- B23 pad 1: Net-(B23-Pad1) -> Net-(B10-Pad1)
- B24 pad 1: Net-(B24-Pad1) -> Net-(B10-Pad1)
- B25 pad 1: Net-(B25-Pad1) -> Net-(B103-Pad1)
- B26 pad 1: Net-(B26-Pad1) -> Net-(B103-Pad1)
- B27 pad 1: Net-(B27-Pad1) -> Net-(B1-Pad1)
- B28 pad 1: Net-(B28-Pad1) -> Net-(B106-Pad1)
- B29 pad 1: Net-(B29-Pad1) -> Net-(B106-Pad1)
- B3 pad 1: Net-(B3-Pad1) -> Net-(B106-Pad1)
- B30 pad 1: Net-(B30-Pad1) -> Net-(B108-Pad1)
- B31 pad 1: Net-(B31-Pad1) -> Net-(B108-Pad1)
- B32 pad 1: Net-(B32-Pad1) -> Net-(B110-Pad1)
- B33 pad 1: Net-(B33-Pad1) -> Net-(B110-Pad1)
- B34 pad 1: Net-(B34-Pad1) -> Net-(B100-Pad1)
- B35 pad 1: Net-(B35-Pad1) -> Net-(B100-Pad1)
- B36 pad 1: Net-(B36-Pad1) -> Net-(B10-Pad1)
- B37 pad 1: Net-(B37-Pad1) -> Net-(B10-Pad1)
- B38 pad 1: Net-(B38-Pad1) -> Net-(B103-Pad1)
- B39 pad 1: Net-(B39-Pad1) -> Net-(B103-Pad1)
- B4 pad 1: Net-(B4-Pad1) -> Net-(B108-Pad1)
- B5 pad 1: Net-(B5-Pad1) -> Net-(B108-Pad1)
- B6 pad 1: Net-(B6-Pad1) -> Net-(B110-Pad1)
- B7 pad 1: Net-(B7-Pad1) -> Net-(B110-Pad1)
- B8 pad 1: Net-(B8-Pad1) -> Net-(B100-Pad1)
- B9 pad 1: Net-(B9-Pad1) -> Net-(B100-Pad1)
- F1 pad 2: Net-(F1-Pad2) -> Net-(B1-Pad1)
- F2 pad 2: Net-(F10-Pad2) -> Net-(B106-Pad1)
- F3 pad 2: Net-(F11-Pad1) -> Net-(B108-Pad1)
- F4 pad 2: Net-(F13-Pad1) -> Net-(B110-Pad1)
- F5 pad 2: Net-(F15-Pad1) -> Net-(B100-Pad1)
- F6 pad 2: Net-(F17-Pad1) -> Net-(B10-Pad1)
- F7 pad 2: Net-(F19-Pad1) -> Net-(B103-Pad1)
Routing:
- net Net-(B10-Pad1): track 0.00 -> 540.1 mm
- net Net-(B103-Pad1): track 0.00 -> 457.0 mm
- net Net-(B106-Pad1): track 0.00 -> 420.3 mm
- net Net-(B100-Pad1): track 0.00 -> 388.0 mm
- net Net-(B108-Pad1): track 0.00 -> 385.4 mm
- net Net-(B1-Pad1): track 2.32 -> 387.1 mm
- net Net-(B110-Pad1): track 0.00 -> 353.0 mm
- net Net-(F1-Pad2): track 126.5 -> 0.00 mm
- net BMS2: track 0.00 -> 91.7 mm
- net BSM4: track 0.00 -> 81.9 mm
- net BMS6: track 0.00 -> 72.2 mm
- net BMS8: track 0.00 -> 62.4 mm
- net BMS10: track 0.00 -> 52.6 mm
- net BMS12: track 0.00 -> 42.7 mm
- net BMS14: track 0.00 -> 32.2 mm
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- removed copper zone on F.Cu, net Net-(F11-Pad1)
Other:
- board size 250 x 251 mm -> 260 x 260 mm
- board text added: "1"
- board text added: "10"
- board text added: "11"
- board text added: "12"
- board text added: "13"
- board text added: "14"
- board text added: "2"
- board text added: "3"
- board text added: "4"
- board text added: "5"
- board text added: "6"
- board text added: "7"
- board text added: "8"
- board text added: "9"

Commit message: Changes for v0.1-rc
Parts:
- added REF**: OSHW-Logo2_7.3x6mm_Copper, Symbol:OSHW-Logo2_7.3x6mm_Copper, B.Cu at (198.0, 261.5)
- added REF**: MountingHole_5.3mm_M5_Pad_Via, MountingHole:MountingHole_5.3mm_M5_Pad_Via, F.Cu at (24.2, 260.2)
- added REF**: OSHW-Logo2_7.3x6mm_Copper, Symbol:OSHW-Logo2_7.3x6mm_Copper, F.Cu at (198.0, 261.5)
Routing:
- net Net-(B1-Pad1): track 387.1 -> 383.4 mm, vias 0 -> 2
- net Net-(B103-Pad1): track 457.0 -> 456.2 mm
- net (no net): vias 0 -> 4
Other:
- board text added: "Installation Label"
- board text added: "Positive / Negative"
- board text added: "github.com/mitchese/easypowerwall Release: v0.1-rc"
