File: easypowerwall.kicad_pcb (KiCad board)
At the start: 2 copper layers, 260 x 260 mm, 165 parts, among them J1 Conn_01x14, J2 Conn_01x07

Commit message: Rename project
Parts:
- added REF**: OSHW-Logo2_7.3x6mm_Copper, Symbol:OSHW-Logo2_7.3x6mm_Copper, B.Cu at (198.0, 261.5)
- added REF**: MountingHole_5.3mm_M5_Pad_Via, MountingHole:MountingHole_5.3mm_M5_Pad_Via, F.Cu at (24.2, 260.2)
- added REF**: OSHW-Logo2_7.3x6mm_Copper, Symbol:OSHW-Logo2_7.3x6mm_Copper, F.Cu at (198.0, 261.5)
- added REF**: MountingHole_3.5mm, MountingHole:MountingHole_3.5mm, F.Cu at (213.0, 73.0)
- added REF**: MountingHole_3.5mm, MountingHole:MountingHole_3.5mm, F.Cu at (213.0, 193.0)
- added REF**: MountingHole_3.5mm, MountingHole:MountingHole_3.5mm, F.Cu at (73.0, 193.0)
- added REF**: MountingHole_3.5mm, MountingHole:MountingHole_3.5mm, F.Cu at (73.0, 73.0)
Routing:
- net Net-(B10-Pad1): track 423.6 -> 539.8 mm
- net Net-(B1-Pad1): track 387.1 -> 383.4 mm, vias 0 -> 2
- net Net-(B103-Pad1): track 457.0 -> 456.2 mm
- net (no net): vias 0 -> 4
Other:
- board text added: "Installation Label"
- board text added: "Positive / Negative"
- board text added: "github.com/mitchese/easypowerwall Release: v0.1-rc"
